File: Custom-Keyboard.kicad_pcb (KiCad board)
At the start: 2 copper layers, 406.4 x 117.5 mm, 188 parts, among them SW1 SW_PUSH, U1 ATmega32U4-AU, Y1 16MHz

Commit message: Routing
All components routed and connected to the MCU.
Parts:
- ENTER1: footprint MX_Alps_Hybrid:MX-2U-ReversedStabilizers -> MX_Alps_Hybrid:MX-2U
- moved C6 18.6 mm to (108.0, 53.2), turned to 270 degrees
- moved R4 13.6 mm to (129.4, 53.2)
- moved C2 12.8 mm to (114.3, 38.9)
- moved C7 12.8 mm to (109.5, 47.6)
- moved R3 12.8 mm to (111.1, 38.9), turned to 270 degrees
- moved C3 12.8 mm to (123.8, 57.9)
- moved C4 12.8 mm to (123.0, 34.1)
- moved C5 12.8 mm to (115.1, 34.1)
- moved U1 12.8 mm to (119.9, 48.4)
- moved Y1 12.8 mm to (119.1, 34.1)
- moved C1 12.0 mm to (129.4, 44.5)
- turned F1 to 90 degrees
Connections:
- D19 pad 1: Net-(D19-Pad1) -> Row6
- D21 pad 1: Net-(D19-Pad1) -> Row6
- D22 pad 1: Net-(D19-Pad1) -> Row6
- D25 pad 1: Net-(D25-Pad1) -> Row3
- D30 pad 1: Net-(D30-Pad1) -> Row3
- D35 pad 1: Net-(D35-Pad1) -> Row3
- D40 pad 1: Net-(D40-Pad1) -> Row3
- D44 pad 1: Net-(D44-Pad1) -> Row3
- D48 pad 1: Net-(D48-Pad1) -> Row3
- D52 pad 1: Net-(D52-Pad1) -> Row3
- D57 pad 1: Net-(D57-Pad1) -> Row3
- D61 pad 1: Net-(D61-Pad1) -> Row3
- D65 pad 1: Net-(D65-Pad1) -> Row3
- D69 pad 1: Net-(D69-Pad1) -> Row3
- D74 pad 1: Net-(D74-Pad1) -> Row3
- D81 pad 1: Net-(D81-Pad1) -> Row3
- D85 pad 1: Net-(D85-Pad1) -> Row3
- U1 pad 1: Net-(U1-Pad1) -> Col1
- U1 pad 10: Net-(U1-Pad10) -> Row5
- U1 pad 11: Net-(U1-Pad11) -> Row6
- U1 pad 12: Net-(U1-Pad12) -> Col4
- U1 pad 18: Net-(U1-Pad18) -> Row1
- U1 pad 19: Net-(U1-Pad19) -> Col19
- U1 pad 20: Net-(U1-Pad20) -> Row2
- U1 pad 21: Net-(U1-Pad21) -> Row3
- U1 pad 22: Net-(U1-Pad22) -> Row4
- U1 pad 25: Net-(U1-Pad25) -> Col5
- U1 pad 26: Net-(U1-Pad26) -> Col6
- U1 pad 27: Net-(U1-Pad27) -> Col7
- U1 pad 28: Net-(U1-Pad28) -> Col8
- U1 pad 29: Net-(U1-Pad29) -> Col9
- U1 pad 30: Net-(U1-Pad30) -> Col10
- U1 pad 31: Net-(U1-Pad31) -> Col11
- U1 pad 32: Net-(U1-Pad32) -> Col12
- U1 pad 36: Net-(U1-Pad36) -> Col13
- U1 pad 37: Net-(U1-Pad37) -> Col14
- U1 pad 38: Net-(U1-Pad38) -> Col15
- U1 pad 39: Net-(U1-Pad39) -> Col16
- U1 pad 40: Net-(U1-Pad40) -> Col17
- U1 pad 41: Net-(U1-Pad41) -> Col18
- U1 pad 8: Net-(U1-Pad8) -> Col2
- U1 pad 9: Net-(U1-Pad9) -> Col3
Routing:
- net Row4: track 0.00 -> 533.7 mm, vias 0 -> 2
- net Row3: track 0.00 -> 521.8 mm, vias 0 -> 2
- net Row2: track 0.00 -> 502.7 mm, vias 0 -> 2
- net Row1: track 0.00 -> 431.8 mm, vias 0 -> 2
- net Row5: track 0.00 -> 405.3 mm, vias 0 -> 2
- net Col19: track 0.00 -> 362.4 mm, vias 0 -> 1
- net Col17: track 0.00 -> 351.5 mm, vias 0 -> 3
- net Col18: track 0.00 -> 349.6 mm, vias 0 -> 3
- net Col16: track 0.00 -> 342.7 mm, vias 0 -> 3
- net Col15: track 0.00 -> 338.8 mm, vias 0 -> 3
- net Col14: track 0.00 -> 281.8 mm, vias 0 -> 3
- net Col13: track 0.00 -> 260.7 mm, vias 0 -> 3
- net Col11: track 0.00 -> 229.9 mm, vias 0 -> 3
- net Col12: track 0.00 -> 218.3 mm, vias 0 -> 3
- net Col2: track 0.00 -> 206.8 mm, vias 0 -> 3
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Other:
- net class Default: trace_width 0.25 -> 0.254
- net class Power added: clearance 0.2, trace_width 0.381, via_dia 0.8, via_drill 0.4

Commit message: PCB Size Error Fixing
Noticed a mistake in the PCB side edge going in to a hole for Stabilizers. Made PCB a little tiny bit bigger to compensate.
Parts:
- moved USB1 1.24 mm to (108.0, 20.2)
Routing:
- net VCC: track 10.9 -> 12.1 mm
- net D-: track 5.21 -> 6.45 mm
- net D+: track 5.54 -> 6.78 mm
- net GND: track 152.8 -> 154.0 mm
Other:
- board size 406.4 x 117.5 mm -> 408.9 x 120.1 mm
Changed lines of the file:
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@@
     (thickness 1.6)
     (drawings 8)
-    (tracks 1444)
+    (tracks 1448)
     (zones 0)
     (modules 188)
@@
     (solder_mask_min_width 0.25)
     (aux_axis_origin 0 0)
-    (visible_elements FFFFFF7F)
+    (visible_elements FFFFF77F)
     (pcbplotparams
       (layerselection 0x010fc_ffffffff)
@@
   )
   (module random-keyboard-parts:Molex-0548190589 (layer B.Cu)
-    (at 107.95 21.43125 270)
+    (at 107.95 20.193 270)
     (attr smd)
     (fp_text reference USB1 (at 2.032 0 180) (layer B.SilkS)
@@
     (pad "" np_thru_hole circle (at 11.938 8.255 270) (size 3.9878 3.9878) (drill 3.9878) (layers *.Cu *.Mask))
   )
-  (gr_line (start 428.625 136.525) (end 24.60625 137.31875) (layer Edge.Cuts) (width 0.15))
-  (gr_line (start 429.41875 135.73125) (end 429.41875 21.43125) (layer Edge.Cuts) (width 0.15))
-  (gr_arc (start 428.625 135.73125) (end 428.625 136.525) (angle -90) (layer Edge.Cuts) (width 0.15))
-  (gr_line (start 24.60625 19.84375) (end 427.83125 19.84375) (layer Edge.Cuts) (width 0.15))
-  (gr_line (start 23.01875 135.73125) (end 23.01875 21.43125) (layer Edge.Cuts) (width 0.15))
-  (gr_arc (start 24.60625 135.73125) (end 23.01875 135.73125) (angle -90) (layer Edge.Cuts) (width 0.15))
-  (gr_arc (start 24.60625 21.43125) (end 24.60625 19.84375) (angle -90) (layer Edge.Cuts) (width 0.15))
-  (gr_arc (start 427.83125 21.43125) (end 429.41875 21.43125) (angle -90) (layer Edge.Cuts) (width 0.15))
+  (gr_line (start 429.387 18.542) (end 22.987 18.542) (layer Edge.Cuts) (width 0.15))
+  (gr_line (start 430.657 136.525) (end 430.657 19.812) (layer Edge.Cuts) (width 0.15))
+  (gr_line (start 23.114 138.684) (end 429.387 137.795) (layer Edge.Cuts) (width 0.15))
+  (gr_line (start 21.717 19.812) (end 21.844 137.414) (layer Edge.Cuts) (width 0.15))
+  (gr_arc (start 22.987 19.812) (end 22.987 18.542) (angle -90) (layer Edge.Cuts) (width 0.15))
+  (gr_arc (start 429.387 19.812) (end 430.657 19.812) (angle -90) (layer Edge.Cuts) (width 0.15))
+  (gr_arc (start 429.387 136.525) (end 429.387 137.795) (angle -90) (layer Edge.Cuts) (width 0.15))
+  (gr_arc (start 23.114 137.414) (end 21.844 137.414) (angle -90) (layer Edge.Cuts) (width 0.15))
   (segment (start 149.38375 36.35375) (end 158.90875 45.87875) (width 0.254) (layer F.Cu) (net 3))
   (segment (start 149.38375 26.82875) (end 149.38375 36.35375) (width 0.254) (layer F.Cu) (net 3))
@@
   (segment (start 102.46875 78.05) (end 101.18775 78.05) (width 0.381) (layer B.Cu) (net 20))
   (segment (start 110.49 54.7855) (end 111.2035 55.499) (width 0.381) (layer B.Cu) (net 20))
+  (segment (start 109.55 25.93125) (end 109.55 24.693) (width 0.381) (layer B.Cu) (net 20))
   (segment (start 115.062 55.613) (end 115.85625 54.81875) (width 0.381) (layer B.Cu) (net 21))
   (segment (start 112.255 55.613) (end 115.062 55.613) (width 0.381) (layer B.Cu) (net 21))
@@
   (segment (start 28.73375 61.468) (end 28.73375 62.15875) (width 0.254) (layer F.Cu) (net 131))
   (segment (start 28.73375 45.87875) (end 28.73375 61.468) (width 0.254) (layer F.Cu) (net 131))
+  (segment (start 106.35 25.93125) (end 106.35 24.693) (width 0.381) (layer B.Cu) (net 140))
+  (segment (start 107.95 25.93125) (end 107.95 24.693) (width 0.254) (layer B.Cu) (net 220))
+  (segment (start 107.15 25.93125) (end 107.15 24.693) (width 0.254) (layer B.Cu) (net 221))
   (segment (start 103.24775 129.44375) (end 104.741 130.937) (width 0.254) (layer B.Cu) (net 298))
   (segment (start 102.39375 129.44375) (end 103.24775 129.44375) (width 0.254) (layer B.Cu) (net 298))
