File: Custom-Keyboard.kicad_pcb (KiCad board)
At the start: 2 copper layers, 408.9 x 120.1 mm, 188 parts, among them SW1 SW_PUSH, U1 ATmega32U4-AU, Y1 16MHz

Commit message: Footprint Change - No LEDs
Schematic has LED pads, but since I don't intend to add LEDs to the keyboard just yet, I changed the footprints to not have any. Don't want there to be any confusion.
Parts:
- AKEY1, BKEY1, CBRAC1, CKEY1, CLN1, CMMA1, DEL1, DIV1, DKEY1, DOWN1, EIGHT1, EIGHT2, EKEY1, EQUALS1, ESC1, FIVE1, FIVE2, FKEY1, FOUR1, FOUR2, FSLSH1, GKEY1, HKEY1, IKEY1, JKEY1, KKEY1, LEFT1, LKEY1, MACRO1, MACRO2, MACRO3, MACRO4, MINUS1, MINUS2, MKEY1, MULT1, NINE1, NINE2, NKEY1, NUM1, OBRAC1, OKEY1, ONE1, ONE2, PER1, PKEY1, PLUS1, QKEY1, QUT1, RGHT1, RKEY1, SEVEN1, SEVEN2, SIX1, SIX2, SKEY1, THREE1, THREE2, TILDE1, TKEY1, TWO1, TWO2, UKEY1, UP1, VKEY1, WKEY1, XKEY1, YKEY1, ZERO2, ZKEY1: footprint MX_Alps_Hybrid:MX-1U -> MX_Alps_Hybrid:MXOnly-1U-NoLED
- ALT1, CTRL1, FN1, LOWER1, WIN1: footprint MX_Alps_Hybrid:MX-1.25U -> MX_Alps_Hybrid:MXOnly-1.25U-NoLED
- BACK1, ENTER1, ZERO1: footprint MX_Alps_Hybrid:MX-2U -> MX_Alps_Hybrid:MXOnly-2U-NoLED
- BSLSH1, TAB1: footprint MX_Alps_Hybrid:MX-1.5U -> MX_Alps_Hybrid:MXOnly-1.5U-NoLED
- CAPS1: footprint MX_Alps_Hybrid:MX-1.75U -> MX_Alps_Hybrid:MXOnly-1.75U-NoLED
- ENTER2, SHIFT1: footprint MX_Alps_Hybrid:MX-2.25U -> MX_Alps_Hybrid:MXOnly-2.25U-NoLED
- SHIFT2: footprint MX_Alps_Hybrid:MX-2.75U -> MX_Alps_Hybrid:MXOnly-2.75U-NoLED
- SPC1: footprint MX_Alps_Hybrid:MX-6.25U -> MX_Alps_Hybrid:MXOnly-6.25U-NoLED

Commit message: MASSIVE Mess Up fix
Rebuilt the whole repository from a back up because I screwed up pretty badly when testing USB-C.
Parts:
- RAISE1: footprint MX_Alps_Hybrid:MX-1.25U -> MX_Alps_Hybrid:MXOnly-1.25U-NoLED
